File: WLED Controller.kicad_pcb (KiCad board)
At the start: 2 copper layers, 100 x 100 mm, 85 parts, among them J1 PROG, J10 Ch 4 S1 Start, J11 Ch 5 S1 Start, J12 Ch 6 S1 Start, J13 Ch 7 S1 Start, J14 Ch 2 S1 End, J15 Ch 2 S2 Start, J16 Ch 2 S2 End, J17 Ch 2 S3 Start, J18 Ch 2 S3 End, J19 Ch 2 S4 Start, J2 MAIN OUT, J20 Ch 2 S4 End, J21 Ch 2 S5 Start, J22 Ch 3 S1 End, J23 Ch 3 S2 Start, J24 Ch 3 S2 End, J25 Ch 1 S3 Start, J26 Ch 1 S3 End, J27 Ch 1 S4 Start, J28 Ch 1 S4 End, J29 Ch 0 S1 End, J3 MAIN IN, J30 Ch 0 S2 Start, J31 Ch 0 S2 End, J32 Ch 1 S1 End, J33 Ch 1 S2 Start, J34 Ch 1 S2 End, J35 Ch 4 S1 End, J36 Ch 4 S2 Start, J37 Ch 4 S2 End, J38 Ch 5 S1 End, J39 Ch 5 S2 Start, J4 5V Power, J40 Ch 5 S2 End, J41 Ch 6 S1 End, J42 Ch 6 S2 Start, J43 Ch 6 S2 End, J44 Ch 7 S1 End, J45 Ch 7 S2 Start, J46 Strings Power, J5 Strings Power, J6 Ch 0 S1 Start, J7 Ch 1 S1 Start, J8 Ch 2 S1 Start, J9 Ch 3 S1 Start, K1 SANYOU_SRD_Form_C, SW1 RESET, SW2 BOOT, U1 ESP32-WROOM-32, U2 ULN2803A, U3 AMS1117-3.3, U5 74AHCT125, U6 74AHCT125

Commit message: added github url
Other:
- board text added: "https://github.com/andreashergert1984/wled-controller"
Changed lines of the file:
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@@
 		)
 		(property "Value" "Strings Power"
-			(at 2.54 5.08 0)
+			(at -5.08 -5.08 0)
 			(layer "F.SilkS")
 			(effects
@@
 		)
 	)
+	(gr_text "https://github.com/andreashergert1984/wled-controller"
+		(at 67.945 119.38 0)
+		(layer "F.SilkS")
+		(effects
+			(font
+				(size 1.016 1.016)
+				(thickness 0.254)
+				(bold yes)
+			)
+			(justify left bottom)
+		)
+	)
 	(gr_text "WLED Controller"
-		(at 54.61 118.11 0)
+		(at 54.61 114.935 0)
 		(layer "F.SilkS")
 		(effects
@@
 		(name "$teardrop_padvia$")
 		(hatch full 0.1)
-		(priority 30003)
+		(priority 30001)
 		(attr
 			(teardrop
@@
 		(polygon
 			(pts
-				(xy 42.946409 63.095421) (xy 43.395421 62.646409) (xy 42.186704 61.711966) (xy 40.345593 62.446793)
-				(xy 41.889338 63.689736)
+				(xy 37.172047 62.344315) (xy 37.621058 62.793326) (xy 38.65863 63.517477) (xy 40.347007 62.446793)
+				(xy 38.59428 61.518428)
 			)
 		)
@@
 		(name "$teardrop_padvia$")
 		(hatch full 0.1)
-		(priority 30001)
+		(priority 30002)
 		(attr
 			(teardrop
@@
 		(polygon
 			(pts
-				(xy 37.172047 62.344315) (xy 37.621058 62.793326) (xy 38.65863 63.517477) (xy 40.347007 62.446793)
-				(xy 38.59428 61.518428)
+				(xy 43.315028 62.4205) (xy 43.315028 62.0395) (xy 41.992389 61.32419) (xy 40.3453 62.4475) (xy 42.124203 63.319893)
 			)
 		)
@@
 		(name "$teardrop_padvia$")
 		(hatch full 0.1)
-		(priority 30002)
+		(priority 30000)
 		(attr
 			(teardrop
@@
 		(polygon
 			(pts
-				(xy 43.315028 62.4205) (xy 43.315028 62.0395) (xy 41.992389 61.32419) (xy 40.3453 62.4475) (xy 42.124203 63.319893)
+				(xy 42.57 60.120862) (xy 41.3 60.120862) (xy 40.487437 60.467857) (xy 40.3463 62.4485) (xy 42.135807 61.600515)
 			)
 		)
@@
 		(name "$teardrop_padvia$")
 		(hatch full 0.1)
-		(priority 30000)
+		(priority 30003)
 		(attr
 			(teardrop
@@
 		(polygon
 			(pts
-				(xy 42.57 60.120862) (xy 41.3 60.120862) (xy 40.487437 60.467857) (xy 40.3463 62.4485) (xy 42.135807 61.600515)
+				(xy 42.946409 63.095421) (xy 43.395421 62.646409) (xy 42.186704 61.711966) (xy 40.345593 62.446793)
+				(xy 41.889338 63.689736)
 			)
 		)
 	)
 	(zone
-		(net 1)
-		(net_name "+5V")
+		(net 13)
+		(net_name "LINE")
 		(layer "B.Cu")
 		(name "$teardrop_padvia$")
 		(hatch full 0.1)
-		(priority 30000)
+		(priority 30003)
 		(attr
 			(teardrop
@@
 		(polygon
 			(pts
-				(xy 38.684813 59.887987) (xy 37.786787 60.786013) (xy 38.419936 61.935349) (xy 40.347007 62.448207)
-				(xy 39.844606 60.531592)
+				(xy 29.8053 91.208143) (xy 31.0753 91.208143) (xy 31.4403 89.939044) (xy 30.4403 88.2275) (xy 29.4403 89.939044)
 			)
 		)
 	)
 	(zone
-		(net 7)
-		(net_name "NEUT")
+		(net 1)
+		(net_name "+5V")
 		(layer "B.Cu")
 		(name "$teardrop_padvia$")
 		(hatch full 0.1)
-		(priority 30002)
+		(priority 30000)
 		(attr
 			(teardrop
@@
 		(polygon
 			(pts
-				(xy 24.6237 91.208143) (xy 25.8937 91.208143) (xy 26.2587 89.939044) (xy 25.2587 88.2275) (xy 24.2587 89.939044)
+				(xy 38.684813 59.887987) (xy 37.786787 60.786013) (xy 38.419936 61.935349) (xy 40.347007 62.448207)
+				(xy 39.844606 60.531592)
 			)
 		)
 	)
 	(zone
-		(net 13)
-		(net_name "LINE")
+		(net 1)
+		(net_name "+5V")
 		(layer "B.Cu")
 		(name "$teardrop_padvia$")
 		(hatch full 0.1)
-		(priority 30003)
+		(priority 30001)
 		(attr
 			(teardrop
@@
 		(polygon
 			(pts
-				(xy 29.8053 91.208143) (xy 31.0753 91.208143) (xy 31.4403 89.939044) (xy 30.4403 88.2275) (xy 29.4403 89.939044)
+				(xy 38.684813 59.887987) (xy 37.786787 60.786013) (xy 38.419936 61.935349) (xy 40.347007 62.448207)
+				(xy 39.844606 60.531592)
 			)
 		)
 	)
 	(zone
-		(net 2)
-		(net_name "GND")
+		(net 7)
+		(net_name "NEUT")
 		(layer "B.Cu")
-		(hatch edge 0.5)
-		(connect_pads
-			(clearance 0.5)
+		(name "$teardrop_padvia$")
+		(hatch full 0.1)
+		(priority 30002)
+		(attr
+			(teardrop
+				(type padvia)
+			)
 		)
-		(min_thickness 0.25)
+		(connect_pads yes
+			(clearance 0)
+		)
+		(min_thickness 0.0254)
 		(filled_areas_thickness no)
 		(fill yes
 			(thermal_gap 0.5)
 			(thermal_bridge_width 0.5)
+			(island_removal_mode 1)
+			(island_area_min 10)
 		)
 		(polygon
 			(pts
-				(xy 46.355 31.75) (xy 75.565 31.75) (xy 75.565 20.32) (xy 119.38 20.32) (xy 119.38 119.38) (xy 52.07 119.38)
-				(xy 52.07 93.98) (xy 40.005 93.98) (xy 40.005 83.82) (xy 20.32 83.82) (xy 20.32 20.32) (xy 46.355 20.32)
+				(xy 24.6237 91.208143) (xy 25.8937 91.208143) (xy 26.2587 89.939044) (xy 25.2587 88.2275) (xy 24.2587 89.939044)
 			)
 		)
 	)
 	(zone
-		(net 1)
-		(net_name "+5V")
+		(net 2)
+		(net_name "GND")
 		(layer "B.Cu")
-		(name "$teardrop_padvia$")
-		(hatch full 0.1)
-		(priority 30001)
-		(attr
-			(teardrop
-				(type padvia)
-			)
-		)
-		(connect_pads yes
-			(clearance 0)
+		(hatch edge 0.5)
+		(connect_pads
+			(clearance 0.5)
 		)
-		(min_thickness 0.0254)
+		(min_thickness 0.25)
 		(filled_areas_thickness no)
 		(fill yes
 			(thermal_gap 0.5)
 			(thermal_bridge_width 0.5)
-			(island_removal_mode 1)
-			(island_area_min 10)
 		)
 		(polygon
 			(pts
-				(xy 38.684813 59.887987) (xy 37.786787 60.786013) (xy 38.419936 61.935349) (xy 40.347007 62.448207)
-				(xy 39.844606 60.531592)
+				(xy 46.355 31.75) (xy 75.565 31.75) (xy 75.565 20.32) (xy 119.38 20.32) (xy 119.38 119.38) (xy 52.07 119.38)
+				(xy 52.07 93.98) (xy 40.005 93.98) (xy 40.005 83.82) (xy 20.32 83.82) (xy 20.32 20.32) (xy 46.355 20.32)
 			)
 		)
